File: wiiu-reg.kicad_sch (KiCad schematic)
At the start: 88 parts, among them IC1 SIC431CED-T1-GE3, IC2 SIC431CED-T1-GE3, IC3 NCP718ASNADJT1G, U1 AP62301Z6-7, U2 AP62301Z6-7, U3 AP62301Z6-7

Commit message: make thing hopefully suck less
Connections:
- net +5V: no longer C20.1, C21.1, C39.1, C40.1, IC1.12 (VDRV), IC1.15 (VDD), IC2.12 (VDRV), IC2.15 (VDD)
- new net: C40.1, IC2.12 (VDRV)
- new net: C39.1, IC2.15 (VDD)
- new net: C20.1, IC1.15 (VDD)
- new net: C21.1, IC1.12 (VDRV)

Commit message: (hopefully) final layout!
Parts:
- added 3v31: 3v3, TestPoint:TestPoint_Pad_2.0x2.0mm, symbol Connector:TestPoint
- added FAN1: 5v, TestPoint:TestPoint_Pad_2.0x2.0mm, symbol Connector:TestPoint
- added GND1: GND, TestPoint:TestPoint_Pad_2.0x2.0mm, symbol Connector:TestPoint
- C21, C40: value 22uF -> 2.2uF
- renumbered TP10 to 1v1, TP9 to 1v25, TP7 to 1v5, TP5 to 3v3, TP2 to 5v1, TP4 to GND2, TP6 to GND3, TP8 to GND4
Connections:
- net +3V3: now also 3v31.1
- net +5V: now also FAN1.1
- net GND: now also GND1.1

Commit message: Complete redesign
Parts:
- removed 1v1: 1v1, TestPoint:TestPoint_Pad_1.5x1.5mm, symbol Connector:TestPoint
- removed 1v25: 1v25, TestPoint:TestPoint_Pad_1.5x1.5mm, symbol Connector:TestPoint
- removed 1v5: 1v5, TestPoint:TestPoint_Pad_2.0x2.0mm, symbol Connector:TestPoint
- removed 3v3, 3v31: 3v3, TestPoint:TestPoint_Pad_2.0x2.0mm, symbol Connector:TestPoint
- removed 5v1, FAN1: 5v, TestPoint:TestPoint_Pad_2.0x2.0mm, symbol Connector:TestPoint
- removed C1, C22, C41: 100nF, Capacitor_SMD:C_0402_1005Metric, symbol Device:C
- removed C10, C11, C12, C13, C14, C15, C17, C18, C24, C25, C30, C31, C32, C33, C34, C35, C36, C37, C43, C44, C6, C7, C8, C9: 22uF, Capacitor_SMD:C_0603_1608Metric, symbol Device:C
- removed C16, C23, C42: 10uF, Capacitor_SMD:C_0805_2012Metric, symbol Device:C
- removed C19, C29, C38, C5: 0.1uF, Capacitor_SMD:C_0402_1005Metric, symbol Device:C
- removed C2, C26, C27, C28, C3, C4: F930J107KBA, wiiu-reg:F930J107KBA, symbol wiiu-reg:F930J107KBA
- removed C20, C39, C45, C46, C47, C48: 1uF, Capacitor_SMD:C_0402_1005Metric, symbol Device:C
- removed C21, C40: 2.2uF, Capacitor_SMD:C_0402_1005Metric, symbol Device:C
- removed GND1, GND2, GND3, GND4, TP3: GND, TestPoint:TestPoint_Pad_2.0x2.0mm, symbol Connector:TestPoint
- removed IC1, IC2: SIC431CED-T1-GE3, SIC431CEDT1GE3, symbol wiiu-reg:SIC431CED-T1-GE3
- removed IC3: NCP718ASNADJT1G, wiiu-reg:NCP718ASNADJT1G, symbol wiiu-reg:NCP718ASNADJT1G
- removed IC4: ~, Package_TO_SOT_SMD:SOT-23-5, symbol wiiu-reg:TCR2EF11,LM(CT_
- removed L1, L4: MPXV1D0840L1R0, wiiu-reg:MPXV1D0840L1R0, symbol wiiu-reg:MPXV1D0840L1R0
- removed L2, L3, L5: 3.3uH, wiiu-reg:INDM4847X300N, symbol Device:L
- removed R1: 6.67k, Resistor_SMD:R_0402_1005Metric, symbol Device:R
- removed R10, R16, R17, R4, R5: 10k, Resistor_SMD:R_0402_1005Metric, symbol Device:R
- removed R11, R3: 100k, Resistor_SMD:R_0402_1005Metric, symbol Device:R
- removed R12: 12k, Resistor_SMD:R_0402_1005Metric, symbol Device:R
- removed R13, R14, R6, R7: 510k, Resistor_SMD:R_0402_1005Metric, symbol Device:R
- removed R15: 8.66k, Resistor_SMD:R_0402_1005Metric, symbol Device:R
- removed R18: 500, Resistor_SMD:R_0402_1005Metric, symbol Device:R
- removed R2: 52.3k, Resistor_SMD:R_0402_1005Metric, symbol Device:R
- removed R8: 31.6k, Resistor_SMD:R_0402_1005Metric, symbol Device:R
- removed R9: 11k, Resistor_SMD:R_0402_1005Metric, symbol Device:R
- removed U1, U2, U3: AP62301Z6-7, wiiu-reg:AP62301Z6-7, symbol PSU:AP62301Z6-7
- added TP2: GND, TestPoint:TestPoint_Pad_2.0x2.0mm, symbol Connector:TestPoint
Connections:
- net GND: now also TP2.1
- no-connect marks 3 -> 0
Other:
- added sheet DRH (DRH.kicad_sch)
- added sheet Low Power (Low Power.kicad_sch)
- added sheet SiC431 1v (SiC431 1v.kicad_sch)
- added sheet SiC431 1v15 (SiC431 1v15.kicad_sch)
- note removed: "Core Regs"
- note removed: "DRH Regs"
- note removed: "Low Power Regs"
- moved on the sheet: TP1
